File: hardware/rocket_datalogger/rocket_datalogger/aux_sensors.kicad_sch (KiCad schematic)
At the start: 7 parts, among them U4 MS5607-02BA, U8 BME280

Commit message: Changed IMU to BNO055
Previous IMU required 1.85V rail
Parts:
- renumbered C16 to C17, C17 to C18, C18 to C19, TP9 to TP5, TP10 to TP6, U8 to U5
Connections:
- net +3.3V: no longer U5.2 (CSB)
- net GND: now also U5.2 (CSB)
- net SCL_3.3V renamed SCL
- net SDA_3.3V renamed SDA
- no-connect marks 0 -> 1

Commit message: fixed minor hardware issues
Parts:
- C19: footprint (none) -> Capacitor_SMD:C_0603_1608Metric
- TP5, TP6: footprint TestPoint:TestPoint_Pad_D1.0mm -> TestPoint:TestPoint_Pad_D2.0mm
Connections:
- net +3.3V: now also U5.2 (CSB); no longer U5.5 (SDO)
- net GND: now also U5.5 (SDO); no longer U5.2 (CSB)
Other:
- moved on the sheet: C17, C18, TP5, TP6, U5

Commit message: Minor revision
Parts:
- renumbered C19 to C17, C17 to C18, C18 to C19
Changed lines of the file:
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@@
 		(dnp no)
 		(fields_autoplaced yes)
-		(property "Reference" "#PWR048"
+		(property "Reference" "#PWR046"
 			(at 78.74 115.57 0)
 			(effects
@@
 			(project "can_datalogger_board"
 				(path "/742f64ac-c4d8-4561-a2a9-e0e3f6f67ce8/439f5b37-3873-4fdf-9d37-42bf545fa021"
-					(reference "#PWR048")
+					(reference "#PWR046")
 					(unit 1)
 				)
@@
 		(dnp no)
 		(fields_autoplaced yes)
-		(property "Reference" "#PWR042"
+		(property "Reference" "#PWR050"
 			(at 97.79 152.4 0)
 			(effects
@@
 			(project ""
 				(path "/742f64ac-c4d8-4561-a2a9-e0e3f6f67ce8/439f5b37-3873-4fdf-9d37-42bf545fa021"
-					(reference "#PWR042")
+					(reference "#PWR050")
 					(unit 1)
 				)
@@
 		(dnp no)
 		(fields_autoplaced yes)
-		(property "Reference" "C19"
+		(property "Reference" "C17"
 			(at 72.39 41.9162 0)
 			(effects
@@
 			(project ""
 				(path "/742f64ac-c4d8-4561-a2a9-e0e3f6f67ce8/439f5b37-3873-4fdf-9d37-42bf545fa021"
-					(reference "C19")
+					(reference "C17")
 					(unit 1)
 				)
@@
 		(dnp no)
 		(fields_autoplaced yes)
-		(property "Reference" "#PWR045"
+		(property "Reference" "#PWR042"
 			(at 57.15 41.91 0)
 			(effects
@@
 			(project ""
 				(path "/742f64ac-c4d8-4561-a2a9-e0e3f6f67ce8/439f5b37-3873-4fdf-9d37-42bf545fa021"
-					(reference "#PWR045")
+					(reference "#PWR042")
 					(unit 1)
 				)
@@
 		(dnp no)
 		(fields_autoplaced yes)
-		(property "Reference" "#PWR047"
+		(property "Reference" "#PWR044"
 			(at 69.85 53.34 0)
 			(effects
@@
 			(project "rocket_datalogger"
 				(path "/742f64ac-c4d8-4561-a2a9-e0e3f6f67ce8/439f5b37-3873-4fdf-9d37-42bf545fa021"
-					(reference "#PWR047")
+					(reference "#PWR044")
 					(unit 1)
 				)
@@
 		(dnp no)
 		(fields_autoplaced yes)
-		(property "Reference" "C18"
+		(property "Reference" "C19"
 			(at 90.17 115.5762 0)
 			(effects
@@
 			(project "can_datalogger_board"
 				(path "/742f64ac-c4d8-4561-a2a9-e0e3f6f67ce8/439f5b37-3873-4fdf-9d37-42bf545fa021"
-					(reference "C18")
+					(reference "C19")
 					(unit 1)
 				)
@@
 		(dnp no)
 		(fields_autoplaced yes)
-		(property "Reference" "#PWR049"
+		(property "Reference" "#PWR047"
 			(at 78.74 171.45 0)
 			(effects
@@
 			(project "can_datalogger_board"
 				(path "/742f64ac-c4d8-4561-a2a9-e0e3f6f67ce8/439f5b37-3873-4fdf-9d37-42bf545fa021"
-					(reference "#PWR049")
+					(reference "#PWR047")
 					(unit 1)
 				)
@@
 		(on_board yes)
 		(dnp no)
-		(property "Reference" "C17"
+		(property "Reference" "C18"
 			(at 69.85 120.6562 0)
 			(effects
@@
 			(project "can_datalogger_board"
 				(path "/742f64ac-c4d8-4561-a2a9-e0e3f6f67ce8/439f5b37-3873-4fdf-9d37-42bf545fa021"
-					(reference "C17")
+					(reference "C18")
 					(unit 1)
 				)
@@
 		(dnp no)
 		(fields_autoplaced yes)
-		(property "Reference" "#PWR043"
+		(property "Reference" "#PWR045"
 			(at 72.39 133.35 0)
 			(effects
@@
 			(project "can_datalogger_board"
 				(path "/742f64ac-c4d8-4561-a2a9-e0e3f6f67ce8/439f5b37-3873-4fdf-9d37-42bf545fa021"
-					(reference "#PWR043")
+					(reference "#PWR045")
 					(unit 1)
 				)
@@
 		(dnp no)
 		(fields_autoplaced yes)
-		(property "Reference" "#PWR046"
+		(property "Reference" "#PWR043"
 			(at 57.15 83.82 0)
 			(effects
@@
 			(project ""
 				(path "/742f64ac-c4d8-4561-a2a9-e0e3f6f67ce8/439f5b37-3873-4fdf-9d37-42bf545fa021"
-					(reference "#PWR046")
+					(reference "#PWR043")
 					(unit 1)
 				)
@@
 		(dnp no)
 		(fields_autoplaced yes)
-		(property "Reference" "#PWR044"
+		(property "Reference" "#PWR048"
 			(at 87.63 127 0)
 			(effects
@@
 			(project "can_datalogger_board"
 				(path "/742f64ac-c4d8-4561-a2a9-e0e3f6f67ce8/439f5b37-3873-4fdf-9d37-42bf545fa021"
-					(reference "#PWR044")
+					(reference "#PWR048")
 					(unit 1)
 				)
@@
 		(dnp no)
 		(fields_autoplaced yes)
-		(property "Reference" "#PWR071"
+		(property "Reference" "#PWR049"
 			(at 107.95 130.81 0)
 			(effects
@@
 			(project "rocket_datalogger"
 				(path "/742f64ac-c4d8-4561-a2a9-e0e3f6f67ce8/439f5b37-3873-4fdf-9d37-42bf545fa021"
-					(reference "#PWR071")
-					(unit 1)
-				)
+					(reference "#PWR049")
+					(unit 1)
+				)
