File: hardware/rocket_datalogger/rocket_datalogger/buck_boost_3v3_output_5V_input.kicad_sch (KiCad schematic)
At the start: 12 parts, among them SW1 SW_SPST

Commit message: Changed IMU to BNO055
Previous IMU required 1.85V rail
Parts:
- renumbered C16 to C14, D3 to D9, R5 to R9
Changed lines of the file:
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@@
 		(dnp no)
 		(fields_autoplaced yes)
-		(property "Reference" "#PWR018"
+		(property "Reference" "#PWR029"
 			(at 160.02 114.3 0)
 			(effects
@@
 			(project "rocket_datalogger"
 				(path "/742f64ac-c4d8-4561-a2a9-e0e3f6f67ce8/6c66699f-236e-4731-b034-8ba482d124c5"
-					(reference "#PWR018")
+					(reference "#PWR029")
 					(unit 1)
 				)
@@
 		(dnp no)
 		(fields_autoplaced yes)
-		(property "Reference" "#PWR040"
+		(property "Reference" "#PWR024"
 			(at 80.01 80.01 0)
 			(effects
@@
 			(project ""
 				(path "/742f64ac-c4d8-4561-a2a9-e0e3f6f67ce8/6c66699f-236e-4731-b034-8ba482d124c5"
-					(reference "#PWR040")
+					(reference "#PWR024")
 					(unit 1)
 				)
@@
 		(dnp no)
 		(fields_autoplaced yes)
-		(property "Reference" "#PWR04"
+		(property "Reference" "#PWR030"
 			(at 167.64 99.06 0)
 			(effects
@@
 			(project "rocket_datalogger"
 				(path "/742f64ac-c4d8-4561-a2a9-e0e3f6f67ce8/6c66699f-236e-4731-b034-8ba482d124c5"
-					(reference "#PWR04")
+					(reference "#PWR030")
 					(unit 1)
 				)
@@
 		(dnp no)
 		(fields_autoplaced yes)
-		(property "Reference" "#PWR02"
+		(property "Reference" "#PWR032"
 			(at 194.31 105.41 0)
 			(effects
@@
 			(project ""
 				(path "/742f64ac-c4d8-4561-a2a9-e0e3f6f67ce8/6c66699f-236e-4731-b034-8ba482d124c5"
-					(reference "#PWR02")
+					(reference "#PWR032")
 					(unit 1)
 				)
@@
 		(dnp no)
 		(fields_autoplaced yes)
-		(property "Reference" "#PWR041"
+		(property "Reference" "#PWR028"
 			(at 132.08 111.76 0)
 			(effects
@@
 			(project "rocket_datalogger"
 				(path "/742f64ac-c4d8-4561-a2a9-e0e3f6f67ce8/6c66699f-236e-4731-b034-8ba482d124c5"
-					(reference "#PWR041")
+					(reference "#PWR028")
 					(unit 1)
 				)
@@
 		(dnp no)
 		(fields_autoplaced yes)
-		(property "Reference" "#PWR020"
+		(property "Reference" "#PWR033"
 			(at 193.04 80.01 0)
 			(effects
@@
 			(project ""
 				(path "/742f64ac-c4d8-4561-a2a9-e0e3f6f67ce8/6c66699f-236e-4731-b034-8ba482d124c5"
-					(reference "#PWR020")
+					(reference "#PWR033")
 					(unit 1)
 				)
@@
 		(dnp no)
 		(fields_autoplaced yes)
-		(property "Reference" "#PWR042"
+		(property "Reference" "#PWR026"
 			(at 120.65 96.52 0)
 			(effects
@@
 			(project "rocket_datalogger"
 				(path "/742f64ac-c4d8-4561-a2a9-e0e3f6f67ce8/6c66699f-236e-4731-b034-8ba482d124c5"
-					(reference "#PWR042")
+					(reference "#PWR026")
 					(unit 1)
 				)
@@
 		(dnp no)
 		(fields_autoplaced yes)
-		(property "Reference" "R5"
+		(property "Reference" "R9"
 			(at 196.85 85.0899 0)
 			(effects
@@
 			(project ""
 				(path "/742f64ac-c4d8-4561-a2a9-e0e3f6f67ce8/6c66699f-236e-4731-b034-8ba482d124c5"
-					(reference "R5")
+					(reference "R9")
 					(unit 1)
 				)
@@
 		(dnp no)
 		(fields_autoplaced yes)
-		(property "Reference" "#PWR032"
+		(property "Reference" "#PWR031"
 			(at 185.42 120.65 0)
 			(effects
@@
 			(project "rocket_datalogger"
 				(path "/742f64ac-c4d8-4561-a2a9-e0e3f6f67ce8/6c66699f-236e-4731-b034-8ba482d124c5"
-					(reference "#PWR032")
+					(reference "#PWR031")
 					(unit 1)
 				)
@@
 		(dnp no)
 		(fields_autoplaced yes)
-		(property "Reference" "C16"
+		(property "Reference" "C14"
 			(at 180.34 83.8262 0)
 			(effects
@@
 			(project "rocket_datalogger"
 				(path "/742f64ac-c4d8-4561-a2a9-e0e3f6f67ce8/6c66699f-236e-4731-b034-8ba482d124c5"
-					(reference "C16")
+					(reference "C14")
 					(unit 1)
 				)
@@
 		(dnp no)
 		(fields_autoplaced yes)
-		(property "Reference" "D3"
+		(property "Reference" "D9"
 			(at 198.12 94.2974 90)
 			(effects
@@
 			(project ""
 				(path "/742f64ac-c4d8-4561-a2a9-e0e3f6f67ce8/6c66699f-236e-4731-b034-8ba482d124c5"
-					(reference "D3")
+					(reference "D9")
 					(unit 1)
 				)
@@
 		(dnp no)
 		(fields_autoplaced yes)
-		(property "Reference" "#PWR022"
+		(property "Reference" "#PWR025"
 			(at 95.25 93.98 0)
 			(effects
@@
 			(project "rocket_datalogger"
 				(path "/742f64ac-c4d8-4561-a2a9-e0e3f6f67ce8/6c66699f-236e-4731-b034-8ba482d124c5"
-					(reference "#PWR022")
+					(reference "#PWR025")
 					(unit 1)
 				)
@@
 		(dnp no)
 		(fields_autoplaced yes)
-		(property "Reference" "#PWR021"
+		(property "Reference" "#PWR027"
 			(at 123.19 114.3 0)
 			(effects
@@
 			(project "rocket_datalogger"
 				(path "/742f64ac-c4d8-4561-a2a9-e0e3f6f67ce8/6c66699f-236e-4731-b034-8ba482d124c5"
-					(reference "#PWR021")
-					(unit 1)
-				)
+					(reference "#PWR027")
+					(unit 1)
+				)

Commit message: fixed minor hardware issues
Parts:
- C11, C12, C13, C14: footprint (none) -> Capacitor_SMD:C_0603_1608Metric
- D9: footprint (none) -> LED_SMD:LED_0603_1608Metric
- R9: footprint (none) -> Resistor_SMD:R_0603_1608Metric
- TP2, TP3, TP4: footprint (none) -> TestPoint:TestPoint_Pad_D2.0mm
Changed lines of the file:
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@@
 			)
 		)
-		(property "Footprint" ""
+		(property "Footprint" "TestPoint:TestPoint_Pad_D2.0mm"
 			(at 190.5 78.74 0)
 			(effects
@@
 			)
 		)
-		(property "Footprint" ""
+		(property "Footprint" "TestPoint:TestPoint_Pad_D2.0mm"
 			(at 111.76 78.74 0)
 			(effects
@@
 			)
 		)
-		(property "Footprint" ""
+		(property "Footprint" "TestPoint:TestPoint_Pad_D2.0mm"
 			(at 190.5 113.03 0)
 			(effects
@@
 			)
 		)
-		(property "Footprint" ""
+		(property "Footprint" "Capacitor_SMD:C_0603_1608Metric"
 			(at 95.25 83.82 0)
 			(effects
@@
 			)
 		)
-		(property "Footprint" ""
+		(property "Footprint" "Resistor_SMD:R_0603_1608Metric"
 			(at 194.31 86.36 0)
 			(effects
@@
 			)
 		)
-		(property "Footprint" ""
+		(property "Footprint" "Capacitor_SMD:C_0603_1608Metric"
 			(at 167.64 85.09 0)
 			(effects
@@
 			)
 		)
-		(property "Footprint" ""
+		(property "Footprint" "Capacitor_SMD:C_0603_1608Metric"
 			(at 120.65 87.63 0)
 			(effects
@@
 			)
 		)
-		(property "Footprint" ""
+		(property "Footprint" "Capacitor_SMD:C_0603_1608Metric"
 			(at 177.8 85.09 0)
 			(effects
@@
 			)
 		)
-		(property "Footprint" ""
+		(property "Footprint" "LED_SMD:LED_0603_1608Metric"
 			(at 194.31 93.98 0)
 			(effects

Commit message: Minor revision
Parts:
- removed SW1: SW_SPST, symbol Switch:SW_SPST
- L1: footprint (none) -> Inductor_SMD:L_Coilcraft_LPS3010
- U2: footprint (none) -> rocket_datalogger:DSK0010A
Connections:
- net +BATT: now also C11.1, TP2.1, U2.5 (VIN)
Changed lines of the file:
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@@
 	(wire
 		(pts
-			(xy 76.2 80.01) (xy 80.01 80.01)
+			(xy 86.36 80.01) (xy 95.25 80.01)
 		)
 		(stroke
@@
 		(pts
 			(xy 160.02 95.25) (xy 157.48 95.25)
-		)
-		(stroke
-			(width 0)
-			(type default)
-		)
-	)
-	(wire
-		(pts
-			(xy 90.17 80.01) (xy 95.25 80.01)
 		)
 		(stroke
@@
 	(symbol
 		(lib_id "power:+BATT")
-		(at 76.2 80.01 90)
+		(at 86.36 80.01 90)
 		(unit 1)
 		(exclude_from_sim no)
@@
 		(fields_autoplaced yes)
 		(property "Reference" "#PWR024"
-			(at 80.01 80.01 0)
+			(at 90.17 80.01 0)
 			(effects
 				(font
@@
 		)
 		(property "Value" "+BATT"
-			(at 72.39 80.0099 90)
+			(at 82.55 80.0099 90)
 			(effects
 				(font
@@
 		)
 		(property "Footprint" ""
-			(at 76.2 80.01 0)
+			(at 86.36 80.01 0)
 			(effects
 				(font
@@
 		)
 		(property "Datasheet" ""
-			(at 76.2 80.01 0)
+			(at 86.36 80.01 0)
 			(effects
 				(font
@@
 		)
 		(property "Description" "Power symbol creates a global label with name \"+BATT\""
-			(at 76.2 80.01 0)
+			(at 86.36 80.01 0)
 			(effects
 				(font
@@
 			)
 		)
-		(property "Footprint" ""
+		(property "Footprint" "Inductor_SMD:L_Coilcraft_LPS3010"
 			(at 146.05 64.77 0)
 			(effects
@@
 	)
 	(symbol
-		(lib_id "Switch:SW_SPST")
-		(at 85.09 80.01 0)
-		(unit 1)
-		(exclude_from_sim no)
-		(in_bom yes)
-		(on_board yes)
-		(dnp no)
-		(fields_autoplaced yes)
-		(property "Reference" "SW1"
-			(at 85.09 73.66 0)
-			(effects
-				(font
-					(size 1.27 1.27)
-				)
-			)
-		)
-		(property "Value" "SW_SPST"
-			(at 85.09 76.2 0)
-			(effects
-				(font
-					(size 1.27 1.27)
-				)
-			)
-		)
-		(property "Footprint" ""
-			(at 85.09 80.01 0)
-			(effects
-				(font
-					(size 1.27 1.27)
-				)
-				(hide yes)
-			)
-		)
-		(property "Datasheet" "~"
-			(at 85.09 80.01 0)
-			(effects
-				(font
-					(size 1.27 1.27)
-				)
-				(hide yes)
-			)
-		)
-		(property "Description" "Single Pole Single Throw (SPST) switch"
-			(at 85.09 80.01 0)
-			(effects
-				(font
-					(size 1.27 1.27)
-				)
-				(hide yes)
-			)
-		)
-		(pin "2"
-		)
-		(pin "1"
-		)
-		(instances
-			(project ""
-				(path "/742f64ac-c4d8-4561-a2a9-e0e3f6f67ce8/6c66699f-236e-4731-b034-8ba482d124c5"
-					(reference "SW1")
-					(unit 1)
-				)
-			)
-		)
-	)
-	(symbol
 		(lib_id "Device:R_Small")
 		(at 194.31 86.36 0)
@@
 			)
 		)
-		(property "Footprint" ""
+		(property "Footprint" "rocket_datalogger:DSK0010A"
 			(at 146.05 85.09 0)
 			(effects
