File: hardware/rocket_datalogger/rocket_datalogger/stm32f042k6ux.kicad_sch (KiCad schematic)
At the start: 22 parts, among them J2 TC2030, U1 STM32F042K6Ux, Y1 ECS-160-10-36Q-AES-TR

Commit message: Changed IMU to BNO055
Previous IMU required 1.85V rail
Parts:
- renumbered C3 to C1, C1 to C2, C2 to C3, D1 to D7, D2 to D8, J2 to J3, R1 to R5, R2 to R6, R6 to R8
Connections:
- net GPS_RESET: now also U1.6 (PA0)
- net GPS_TIMEPULSE: now also U1.7 (PA1)
- net SCL: now also U1.19 (PA9)
- net SDA: now also U1.20 (PA10)
- net UART_RX: now also U1.29 (PB6)
- net UART_TX: now also U1.30 (PB7)
- net USB_D_N: now also U1.21 (PA11)
- net USB_D_P: now also U1.22 (PA12)
- net GPIO_1: now reaches U1.10 (PA4)
- net GPIO_2: now reaches U1.11 (PA5)
- net GPIO_3: now reaches U1.12 (PA6)
- net GPIO_4: now reaches U1.13 (PA7)
- net GPIO_5: now reaches U1.18 (PA8)
- net ~IMU_RESET: now reaches U1.8 (PA2)
- net GPIO_0: now reaches U1.9 (PA3)
- no-connect marks 11 -> 7
Other:
- note added: "16 Mhz HSE"
- moved on the sheet: C1, C7, C9, R7, R8, Y1

Commit message: fixed minor hardware issues
Parts:
- R7, R8: footprint (none) -> Resistor_SMD:R_0603_1608Metric
Connections:
- net IMU_INT: now reaches U1.25 (PA15)
- no-connect marks 7 -> 6
Changed lines of the file:
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@@
 	)
 	(no_connect
-		(at 227.33 100.33)
-	)
-	(no_connect
 		(at 201.93 100.33)
 	)
@@
 	(wire
 		(pts
+			(xy 227.33 100.33) (xy 229.87 100.33)
+		)
+		(stroke
+			(width 0)
+			(type default)
+		)
+	)
+	(wire
+		(pts
 			(xy 227.33 69.85) (xy 229.87 69.85)
 		)
@@
 		)
 	)
+	(hierarchical_label "IMU_INT"
+		(shape input)
+		(at 229.87 100.33 0)
+		(effects
+			(font
+				(size 1.27 1.27)
+			)
+			(justify left)
+		)
+	)
 	(hierarchical_label "USB_D_N"
 		(shape bidirectional)
@@
 			)
 		)
-		(property "Footprint" ""
+		(property "Footprint" "Resistor_SMD:R_0603_1608Metric"
 			(at 257.81 77.47 0)
 			(effects
@@
 			)
 		)
-		(property "Footprint" ""
+		(property "Footprint" "Resistor_SMD:R_0603_1608Metric"
 			(at 261.62 77.47 0)
 			(effects

Commit message: Minor revision
Connections:
- net +3V3: no longer U1.17 (VDDIO2), U1.5 (VDDA)
- net BOOT0: now also U1.14 (PB0); no longer U1.31 (PF11)
- net GPIO_0: now also U1.10 (PA4); no longer U1.9 (PA3)
- net GPIO_1: now also U1.11 (PA5); no longer U1.10 (PA4)
- net GPIO_2: now also U1.12 (PA6); no longer U1.11 (PA5)
- net GPIO_3: now also U1.13 (PA7); no longer U1.12 (PA6)
- net GPIO_4: now also U1.18 (PA8); no longer U1.13 (PA7)
- net GPIO_5: now also U1.19 (PA9); no longer U1.18 (PA8)
- net GPS_RESET: now also U1.7 (PA1); no longer U1.6 (PA0)
- net GPS_TIMEPULSE: now also U1.8 (PA2); no longer U1.7 (PA1)
- net IMU_INT: no longer U1.25 (PA15)
- net LED_STATUS_1: now also U1.16 (PB2); no longer U1.14 (PB0)
- net LED_STATUS_2: now also U1.26 (PB3); no longer U1.15 (PB1)
- net NRST: no longer U1.4 (NRST)
- net OSC_IN: now also U1.31 (PF11); no longer U1.2 (PF0)
- net OSC_OUT: no longer U1.3 (PF1)
- net SCL: now also U1.20 (PA10); no longer U1.19 (PA9)
- net SDA: now also U1.21 (PA11); no longer U1.20 (PA10)
- net SWCLK: now also U1.25 (PA15); no longer U1.24 (PA14)
- net SWDIO: now also U1.24 (PA14); no longer U1.23 (PA13)
- net UART_RX: now also U1.32 (PB8); no longer U1.29 (PB6)
- net UART_TX: no longer U1.30 (PB7)
- net USB_D_N: now also U1.22 (PA12); no longer U1.21 (PA11)
- net USB_D_P: now also U1.23 (PA13); no longer U1.22 (PA12)
- net ~IMU_RESET: now also U1.9 (PA3); no longer U1.8 (PA2)
Other:
- moved on the sheet: U1
Changed lines of the file:
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@@
 			)
 		)
-		(property "Description" ""
+		(property "Description" "Power symbol creates a global label with name \"+3.3V\""
 			(at 154.94 88.9 0)
 			(effects
@@
 			)
 		)
-		(property "Description" ""
+		(property "Description" "Power symbol creates a global label with name \"GND\" , ground"
 			(at 124.46 177.8 0)
 			(effects
@@
 	)
 	(symbol
-		(lib_name "+3.3V_3")
 		(lib_id "power:+3.3V")
 		(at 212.09 52.07 0)
@@
 			)
 		)
-		(property "Description" ""
+		(property "Description" "Power symbol creates a global label with name \"+3.3V\""
 			(at 212.09 52.07 0)
 			(effects
@@
 			)
 		)
-		(property "Description" ""
+		(property "Description" "Unpolarized capacitor, small symbol"
 			(at 142.24 36.83 0)
 			(effects
@@
 			)
 		)
-		(property "Description" ""
+		(property "Description" "Resistor"
 			(at 143.51 97.79 0)
 			(effects
@@
 	)
 	(symbol
-		(lib_name "+3.3V_2")
 		(lib_id "power:+3.3V")
 		(at 33.02 87.63 0)
@@
 			)
 		)
-		(property "Description" ""
+		(property "Description" "Power symbol creates a global label with name \"+3.3V\""
 			(at 33.02 87.63 0)
 			(effects
@@
 	)
 	(symbol
-		(lib_name "GND_5")
 		(lib_id "power:GND")
 		(at 134.62 177.8 0)
@@
 			)
 		)
-		(property "Description" ""
+		(property "Description" "Power symbol creates a global label with name \"GND\" , ground"
 			(at 134.62 177.8 0)
 			(effects
@@
 			)
 		)
-		(property "Description" ""
+		(property "Description" "Light emitting diode"
 			(at 85.09 104.14 0)
 			(effects
@@
 			)
 		)
+		(property "Sim.Pins" "1=K 2=A"
+			(at 85.09 104.14 0)
+			(effects
+				(font
+					(size 1.27 1.27)
+				)
+			)
+		)
 		(pin "1"
 		)
@@
 	)
 	(symbol
-		(lib_name "+3.3V_4")
 		(lib_id "power:+3.3V")
 		(at 257.81 71.12 0)
@@
 			)
 		)
-		(property "Description" ""
+		(property "Description" "Unpolarized capacitor, small symbol"
 			(at 134.62 173.99 0)
 			(effects
@@
 			)
 		)
-		(property "Description" ""
+		(property "Description" "Four pin crystal, GND on pins 2 and 4, small symbol"
 			(at 129.54 168.91 0)
 			(effects
@@
 	)
 	(symbol
-		(lib_name "GND_8")
 		(lib_id "power:GND")
 		(at 46.99 170.18 0)
@@
 			)
 		)
-		(property "Description" ""
+		(property "Description" "Power symbol creates a global label with name \"GND\" , ground"
 			(at 46.99 170.18 0)
 			(effects
@@
 			)
 		)
-		(property "Datasheet" "http://www.st.com/st-web-ui/static/active/en/resource/technical/document/datasheet/DM00105814.pdf"
+		(property "Datasheet" "https://www.st.com/resource/en/datasheet/stm32f042k6.pdf"
 			(at 214.63 80.01 0)
 			(effects
@@
 			)
 		)
-		(property "Description" ""
+		(property "Description" "STMicroelectronics Arm Cortex-M0 MCU, 32KB flash, 6KB RAM, 48 MHz, 2.0-3.6V, 28 GPIO, UFQFPN32"
 			(at 214.63 80.01 0)
 			(effects
@@
 			)
 		)
-		(property "Description" ""
+		(property "Description" "Unpolarized capacitor, small symbol"
 			(at 132.08 36.83 0)
 			(effects
@@
 			)
 		)
-		(property "Description" ""
+		(property "Description" "Unpolarized capacitor, small symbol"
 			(at 101.6 36.83 0)
 			(effects
@@
 			)
 		)
-		(property "Description" ""
+		(property "Description" "Resistor"
 			(at 137.16 92.71 0)
 			(effects
@@
 			)
 		)
-		(property "Description" ""
+		(property "Description" "Unpolarized capacitor, small symbol"
 			(at 124.46 173.99 0)
 			(effects
@@
 	)
 	(symbol
-		(lib_name "GND_4")
 		(lib_id "power:GND")
 		(at 214.63 107.95 0)
@@
 			)
 		)
-		(property "Description" ""
+		(property "Description" "Power symbol creates a global label with name \"GND\" , ground"
 			(at 214.63 107.95 0)
 			(effects
@@
 	)
 	(symbol
-		(lib_name "GND_3")
 		(lib_id "power:GND")
 		(at 81.28 41.91 0)
@@
 			)
 		)
-		(property "Description" ""
+		(property "Description" "Power symbol creates a global label with name \"GND\" , ground"
 			(at 81.28 41.91 0)
 			(effects
@@
 	)
 	(symbol
-		(lib_name "GND_2")
 		(lib_id "power:GND")
 		(at 76.2 110.49 0)
@@
 			)
 		)
-		(property "Description" ""
+		(property "Description" "Power symbol creates a global label with name \"GND\" , ground"
 			(at 76.2 110.49 0)
 			(effects
@@
 			)
 		)
-		(property "Description" ""
+		(property "Description" "Jumper, 3-pole, both open"
 			(at 33.02 95.25 0)
 			(effects
@@
 			)
 		)
-		(property "Description" ""
+		(property "Description" "Resistor"
 			(at 76.2 95.25 0)
 			(effects
@@
 	)
 	(symbol
-		(lib_name "GND_7")
 		(lib_id "power:GND")
 		(at 127 105.41 0)
@@
 			)
 		)
-		(property "Description" ""
+		(property "Description" "Power symbol creates a global label with name \"GND\" , ground"
 			(at 127 105.41 0)
 			(effects
@@
 			)
 		)
-		(property "Description" ""
+		(property "Description" "Unpolarized capacitor, small symbol"
 			(at 81.28 36.83 0)
 			(effects
@@
 	)
 	(symbol
-		(lib_name "GND_6")
 		(lib_id "power:GND")
 		(at 33.02 102.87 0)
@@
 			)
 		)
-		(property "Description" ""
+		(property "Description" "Power symbol creates a global label with name \"GND\" , ground"
 			(at 33.02 102.87 0)
 			(effects
@@
 			)
 		)
-		(property "Description" ""
+		(property "Description" "Resistor"
 			(at 85.09 95.25 0)
 			(effects
@@
 	)
 	(symbol
-		(lib_name "LED_1")
 		(lib_id "Device:LED")
 		(at 76.2 104.14 90)
@@
 			)
 		)
-		(property "Description" ""
+		(property "Description" "Light emitting diode"
+			(at 76.2 104.14 0)
+			(effects
+				(font
+					(size 1.27 1.27)
+				)
+			)
+		)
+		(property "Sim.Pins" "1=K 2=A"
 			(at 76.2 104.14 0)
 			(effects
@@
 			)
 		)
-		(property "Description" ""
+		(property "Description" "Unpolarized capacitor, small symbol"
 			(at 46.99 165.1 0)
 			(effects
@@
 			)
 		)
-		(property "Description" ""
+		(property "Description" "Unpolarized capacitor, small symbol"
 			(at 91.44 36.83 0)
 			(effects
@@
 			)
 		)
-		(property "Description" ""
+		(property "Description" "Generic connector, single row, 01x06, script generated (kicad-library-utils/schlib/autogen/connector/)"
 			(at 118.11 95.25 0)
 			(effects
@@
 	)
 	(symbol
-		(lib_name "GND_1")
 		(lib_id "power:GND")
 		(at 134.62 161.29 0)
@@
 			)
 		)
-		(property "Description" ""
+		(property "Description" "Power symbol creates a global label with name \"GND\" , ground"
 			(at 134.62 161.29 0)
 			(effects
@@
 			)
 		)
-		(property "Description" ""
+		(property "Description" "Unpolarized capacitor, small symbol"
 			(at 111.76 36.83 0)
 			(effects
@@
 			)
 		)
-		(property "Description" ""
+		(property "Description" "Unpolarized capacitor, small symbol"
 			(at 121.92 36.83 0)
 			(effects
@@
 	)
 	(symbol
-		(lib_name "+3.3V_1")
 		(lib_id "power:+3.3V")
 		(at 81.28 31.75 0)
@@
 			)
 		)
-		(property "Description" ""
+		(property "Description" "Power symbol creates a global label with name \"+3.3V\""
 			(at 81.28 31.75 0)
 			(effects

Commit message: PCB design rev 1
Connections:
- net +3V3 is gone; now on net +3.3V: C10.1, C2.1, C3.1, C4.1, C5.1, C6.1, C8.1, J3.1 (Pin_1), JP1.3 (B), U1.1 (VDD)
- net +3.3V: now also U1.17 (VDDIO2), U1.5 (VDDA)
- net BOOT0: now also U1.31 (PF11); no longer U1.14 (PB0)
- net GPIO_0: now also U1.9 (PA3); no longer U1.10 (PA4)
- net GPIO_1: now also U1.10 (PA4); no longer U1.11 (PA5)
- net GPIO_2: now also U1.11 (PA5); no longer U1.12 (PA6)
- net GPIO_3: now also U1.12 (PA6); no longer U1.13 (PA7)
- net GPIO_4: now also U1.13 (PA7); no longer U1.18 (PA8)
- net GPIO_5: now also U1.16 (PB2); no longer U1.19 (PA9)
- net GPS_RESET: now also U1.27 (PB4); no longer U1.7 (PA1)
- net GPS_TIMEPULSE: now also U1.28 (PB5); no longer U1.8 (PA2)
- net IMU_INT: now also U1.25 (PA15)
- net LED_STATUS_1: now also U1.14 (PB0); no longer U1.16 (PB2)
- net LED_STATUS_2: now also U1.15 (PB1); no longer U1.26 (PB3)
- net NRST: now also U1.4 (NRST)
- net OSC_IN: now also U1.2 (PF0); no longer U1.31 (PF11)
- net OSC_OUT: now also U1.3 (PF1)
- net SCL: now also U1.19 (PA9); no longer U1.20 (PA10)
- net SDA: now also U1.20 (PA10); no longer U1.21 (PA11)
- net SWCLK: now also U1.24 (PA14); no longer U1.25 (PA15)
- net SWDIO: now also U1.23 (PA13); no longer U1.24 (PA14)
- net USB_D_N: now also U1.21 (PA11); no longer U1.22 (PA12)
- net USB_D_P: now also U1.22 (PA12); no longer U1.23 (PA13)
- net ~IMU_RESET: now also U1.26 (PB3); no longer U1.9 (PA3)
- net UART_MCU_TX: now reaches U1.29 (PB6)
- net UART_MCU_RX: now reaches U1.30 (PB7)
- net UART_RX: no longer names the net of U1.32 (PB8)
Other:
- moved on the sheet: R7, R8
